Commit message: Initial commit for wheelchair_robot

File: wheelchair_robot_description/urdf/wheelchair_robot.urdf (robot description, URDF)
Before this commit: robot wheelchair_robot, 5 links, 4 joints
Links:
- removed link base_scan
- added link laser_frame
Joints:
- joint cam_joint: origin xyz=0.04355 0.0 0.17945 rpy=0.0 0.0 0.0 -> xyz=-0.13 0.0 0.26145 rpy=0.0 0.0 -0.01745
- joint scan_joint: child base_scan -> laser_frame; origin xyz=-0.005 0.0 0.1105 rpy=0.0 0.0 0.0 -> xyz=-0.13 0.0 0.26145 rpy=0.0 0.0 -0.01745
